File: pcb/gate/Gate Controller/RaspberryBox.kicad_sch (KiCad schematic)
At the start: 33 parts, among them J13 AUX, J14 AUX, J15 Conn_01x04_Female, J16 Conn_01x02_Female, J17 AUX, J18 Power, J19 Fiber Power, J20 Driveway lights, J21 POE Camera, J22 Conn_01x08_Female, J23 Right Post, J24 Conn_01x08_Female, J25 Motor Controller, J26 Ethernet, K1 EC2-5SNU, P1 pi, Q3 FDC6561AN, T1 STD40NF10

Commit message: latest updates
Parts:
- removed J22, J24: Conn_01x08_Female, symbol Connector:Conn_01x08_Female
- removed J23: Right Post, Connector_JST:JST_XH_PinSWAP, symbol Connector:Conn_01x08_Male
- removed J25: Motor Controller, Connector_JST:JST_XH_PinSWAP, symbol Connector:Conn_01x08_Male
- added J20, J21: RJ45_Shielded, Connector_RJ:RJ45_Amphenol_RJHSE5380, symbol Connector:RJ45_Shielded
- added U2: ~, Logos:QRCode Github Automation, symbol Graphic:QR_Automation
- J11: renamed from J13; footprint TerminalBlock_Phoenix:TerminalBlock_Phoenix_PT_1.5-8-PVH-3.5 -> TerminalBlock_Phoenix:TerminalBlock_Phoenix_PT-1,5-8-3.5-H_1x08_P3.50mm_Horizontal
- renumbered J14 to J12, J15 to J13, J16 to J14, J17 to J15, J18 to J16, J19 to J17, J20 to J18, J21 to J19, J26 to J22
Connections:
- net GATE_LED_12V is gone; now on net GND: T1.3 (S)
- net +12V: now also J20.1, J21.1; no longer J17.1 (Pin_1), J17.3 (Pin_3), T1.2 (D)
- net +3V3: now also J20.8, J21.8
- net +5V: now also J17.1 (Pin_1), J17.3 (Pin_3)
- net CN1_24v(FL): now also J20.3, J21.3
- net GND: now also J20.6, J20.SH, J21.6, J21.SH
- net REED LEFT: now also J21.7
- net REED RIGHT: now also J20.7
- net SCL1: now also J21.4
- net SDA1: now also J21.5
- net at K1.1: now also J12.3 (Pin_3); no longer J12.2 (Pin_2)
- net at K1.12: now also J12.2 (Pin_2); no longer J12.3 (Pin_3)
- new net GATE_LED_COM: J20.2, J21.2, T1.2 (D)
- no-connect marks 29 -> 27
Other:
- moved on the sheet: J12, K1

Commit message: reworked to add i2c pullups and reduces unusedd components
Parts:
- removed R11, R12: 1K, Resistor_SMD:R_1206_3216Metric, symbol Device:R
- R10, R9: value 10K -> 1.8K
- renumbered J14 to J10, J15 to J11, J16 to J12, J17 to J13, J18 to J14, J19 to J15, J20 to J16, J21 to J17, J22 to J18, J11 to J7, J12 to J8, J13 to J9
Connections:
- net REED LEFT is gone; now on net GND: J17.7
- net +3V3: now also J17.6, R10.2, R9.2; no longer J16.8, J17.8
- net GND: now also J17.5; no longer J17.6, R10.1, R9.1
- net Rpi11: now also Q3.1, R8.1; no longer T1.1 (G)
- net Rpi15: no longer R10.2
- net Rpi16: no longer R9.2
- net SCL1: now also R9.1
- net SDA1: now also J17.8, R10.1; no longer J17.5
- net Rpi37: now reaches P1.37 (Pin_37)
- net Rpi37: now also T1.1 (G)
- net REED RIGHT: no longer names the net of J16.7
- removed net Rpi29: P1.29 (Pin_29), Q3.1, R8.1
- no-connect marks 27 -> 28
Other:
- note added: "Twisted pairs"
- note added: "i2c Pullups"
- note removed: "Open/Close Detection"

Commit message: Update with latest changes to fix comms issues
Parts:
- J12, J13, J14: footprint TerminalBlock_TE-Connectivity:TerminalBlock_TE_282834-4_1x04_P2.54mm_Horizontal -> Connector_JST:JST_EH_S4B-EH_1x04_P2.50mm_Horizontal
- P1: footprint Connector_PinSocket_2.54mm:PinSocket_2x20_P2.54mm_Vertical -> Connector_PinSocket_2.54mm:PinSocket_2x10_P2.54mm_Vertical_SMD; symbol Connector_Generic:Conn_02x20_Odd_Even -> Connector_Generic:Raspbery Pi Short 2x10 (top-half)
Connections:
- net GND: no longer P1.25 (Pin_25), P1.30 (Pin_30), P1.34 (Pin_34), P1.39 (Pin_39)
- net Rpi13: now also T1.1 (G)
- net Rpi15: no longer names the net of P1.15 (Pin_15)
- net Rpi16: no longer names the net of P1.16 (Pin_16)
- removed net Rpi37: P1.37 (Pin_37), T1.1 (G)
- no-connect marks 28 -> 15
